File: Frida_printer_board/Frida_printer_board.kicad_sch (KiCad schematic)
At the start: 0 parts

Commit message: input 5v convert
Parts:
- added C?: 10uF 50V, Capacitor_SMD:CP_Elec_6.3x5.9, symbol Device:C_Polarized
- added C?: 100nF, Capacitor_SMD:C_0603_1608Metric, symbol Device:C
- added J?: DCIN, TerminalBlock:TerminalBlock_Altech_AK300-2_P5.00mm, symbol Connector:Screw_Terminal_01x02
- added R? (x2): 100k, Resistor_SMD:R_0603_1608Metric, symbol Device:R
- added R?: 24.9k, Resistor_SMD:R_0603_1608Metric, symbol Device:R
- added U?: MP1584EN, monolitich:SOIC127P600X170-9N, symbol monolitich:MP1584EN
Connections:
- new net: R?.1, R?.2, U?.2 (EN)
- new net: R?.1, U?.6 (FREQ)
- new net: C?.2, U?.1 (SW)
- new net: C?.1, U?.8 (BST)
- new net GND: C?.2, J?.1 (Pin_1), R?.2, R?.2, U?.5 (GND), U?.9 (GND)
- new net VIN: C?.1, J?.2 (Pin_2), R?.1, U?.7 (VIN)
